Commit message: setup gazebo sim

File: description/hardware/robot_core.xacro (robot description, xacro)
@@ -38,4 +38,6 @@
         <origin xyz="0 ${wheel_offset_y} 0" rpy="-${pi/2} 0 0" />
         <axis xyz="0 0 1"/>
+        <limit effort="500.0" velocity="10"/>
+        <dynamics damping="1.0" friction="1.0"/>
     </joint>
     <link name="left_wheel">
@@ -64,4 +66,6 @@
         <origin xyz="0 ${-wheel_offset_y} 0" rpy="${pi/2} 0 0" />
         <axis xyz="0 0 -1"/>
+        <limit effort="500.0" velocity="10"/>
+        <dynamics damping="1.0" friction="1.0"/>
     </joint>
     <link name="right_wheel">

File: description/hardware/robot_description.urdf.xacro (robot description, xacro)
@@ -2,3 +2,4 @@
 <robot xmlns:xacro="http://www.ros.org/wiki/xacro" name="robot">
     <xacro:include filename="robot_core.xacro"/>
+    <xacro:include filename="$(find autonomous_diff_bot)/description/gazebo/robot.gazebo"/>
 </robot>
