Commit message: attempt to fix  hardware description files

File: src/ros2_ws/description/hardware/robot_core.xacro (robot description, xacro)
@@ -1,4 +1,5 @@
 <?xml version="1.0"?>
 <robot xmlns:xacro="http://www.ros.org/wiki/xacro">
+    <xacro:macro name="diffbot" params="prefix"/>
     <xacro:include filename="inertial_macros.xacro"/>
     <xacro:include filename="robot_definitions.xacro"/>

File: src/ros2_ws/description/hardware/robot_description.urdf.xacro (robot description, xacro)
@@ -1,5 +1,11 @@
 <?xml version="1.0"?>
 <robot xmlns:xacro="http://www.ros.org/wiki/xacro" name="robot">
+    <xacro:arg name="prefix" default="" />
+    <xacro:arg name="use_mock_hardware" default="false" />
     <xacro:include filename="robot_core.xacro"/>
-    <xacro:include filename="$(find autonomous_diff_bot)/description/gazebo/robot.gazebo"/>
+    <xacro:include filename="$(find autonomous_diff_bot)/description/ros2_control/diff_bot.ros2_control.xacro"/>
+    <!-- <xacro:include filename="$(find autonomous_diff_bot)/description/gazebo/robot.gazebo"/> -->
+    <xacro:diffbot prefix="$(arg prefix)" />
+    <xacro:diffbot_ros2_control
+        name="DiffBot" prefix="$(arg prefix)" use_mock_hardware="$(arg use_mock_hardware)"/>
 </robot>

File: src/ros2_ws/description/ros2_control/diff_bot.ros2_control.xacro (robot description, xacro)
@@ -1,5 +1,5 @@
 <?xml version="1.0"?>
 <robot xmlns:xacro="http://www.ros.org/wiki/xacro">
-  <xacro:macro name="diffbot_ros2_control" params="name use_mock_hardware">
+  <xacro:macro name="diffbot_ros2_control" params="name prefix use_mock_hardware">
     <ros2_control name="${name}" type="system">
       <xacro:unless value="${use_mock_hardware}">

Commit message: first working communication
Use libdevserial

File: src/ros2_ws/description/hardware/robot_core.xacro (robot description, xacro)
@@ -39,5 +39,5 @@
         <origin xyz="0 ${wheel_offset_y} 0" rpy="-${pi/2} 0 0" />
         <axis xyz="0 0 1"/>
-        <limit effort="500.0" velocity="10"/>
+        <limit effort="500.0" velocity="0"/>
         <dynamics damping="1.0" friction="1.0"/>
     </joint>
@@ -67,5 +67,5 @@
         <origin xyz="0 ${-wheel_offset_y} 0" rpy="${pi/2} 0 0" />
         <axis xyz="0 0 -1"/>
-        <limit effort="500.0" velocity="10"/>
+        <limit effort="500.0" velocity="0"/>
         <dynamics damping="1.0" friction="1.0"/>
     </joint>
